File: macromouse.sch (EAGLE design)
At the start: 61 parts, among them Q1 BS170, Q2 BS170, Q3 BS170, Q7 BS170, Q8 BS170, Q9 BS170

Commit message: Updated Schematic: all parts are smd and have the correct pins
still need to choose resis/cap values and figure out boot push button
Parts:
- removed 1.8K, 1.8K1, 1.8K2, 1.8K3, 1.8K4, 1.8K5: (no value), SparkFun:RESISTOR0402-RES
- removed JP2: (no value), SparkFun:M06LOCK
- added C17: 0.1uF, SparkFun:CAP0603-CAP
- added IRE1: EMITTER, sfh4550 _ teft4300:EMITTER
- added R13, R14, R15, R16, R17, R19: (no value), SparkFun:RESISTOR0603-RES
- added S2: (no value), SparkFun:TAC_SWITCHPTH
- added SERIAL: (no value), pinhead:PINHD-1X2
- added SW: (no value), pinhead:PINHD-1X3
- C1: value 0.1uF -> (none)
- C10, C11, C12, C13, C14, C15, C16, C5, C6, C7, C8, C9: device SparkFun-Capacitors:CAPEZ -> SparkFun:CAP0603-CAP
- C2: device SparkFun:CAP0402-CAP -> SparkFun:CAP0603-CAP
- C3: value 10uF -> (none)
- ENCODER: device SparkFun:M06LOCK -> pinhead:PINHD-2X6
- HBRIDGE: value L293D -> L293DD; device st-microelectronics:L293D -> st-microelectronics:L293DD
- R1, R2, R3, R4, R5, R6: value (none) -> 1.8k; device SparkFun-Passives:RESISTORAXIAL-0.3 -> SparkFun:RESISTOR0603-RES
- R10, R11, R12, R7, R8, R9: device SparkFun-Passives:RESISTORAXIAL-0.3 -> SparkFun:RESISTOR0603-RES
- S1: device SparkFun-Electromechanical:SWITCH-SPDTPTH -> SparkFun:TAC_SWITCHPTH
- U$4: value EMITTER -> TS02_SWITCH; device sfh4550 _ teft4300:EMITTER -> 2.54mm slide switch:TS02_SWITCH
- renumbered U$10 to IRE5, U$11 to IRE6, U$6 to IRE2, U$7 to IRE3, U$8 to IRE4
Connections:
- removed net BATT: HBRIDGE.VCC2
- removed net BW_NUCLEO: HBRIDGE.2A, HBRIDGE.3A
- removed net FW_NUCLEO: HBRIDGE.1A, HBRIDGE.4A
- removed net N$8: HBRIDGE.GND2
- removed net NUCLEO: ENCODER.2, ENCODER.3, JP2.2, JP2.3, Q8.G, Q9.G, R10.2, R12.2
- removed net PA0: 1.8K.2, Q4.E
- removed net PA15: Q3.G, R6.2
- removed net PA4: 1.8K1.2, Q5.E
- removed net PB7: Q7.G, R8.2
- removed net PC0: 1.8K2.2, Q6.E
- removed net PC1: 1.8K3.2, Q10.E
- removed net PC10: Q1.G, R2.2
- removed net PC11: Q2.G, R4.2
- removed net PC2: 1.8K4.2, Q11.E
- removed net PC3: 1.8K5.2, Q12.E
- new net ASDF: S2.3
- new net BOOT: S2.1, U$9.PB2
- new net N$13: HBRIDGE.EN1
- new net NRST: S1.1, U$9.NRST
- new net PA_0: Q4.E, R1.2, U$9.PA0_AKUP
- new net PA_1: ENCODER.8, U$9.PA1
- new net PA_10: SERIAL.2, U$9.PA10
- new net PA_11: Q9.G, R8.2, U$9.PA11
- new net PA_13: SW.2, U$9.PA13
- new net PA_14: SW.3, U$9.PA14
- new net PA_15: ENCODER.5, U$9.PA15
- new net PA_3: Q3.G, R14.2, U$9.PA3
- new net PA_4: Q5.E, R2.2, U$9.PA4
- new net PA_5: Q7.G, R11.2, U$9.PA5
- new net PA_6: Q2.G, R16.2, U$9.PA6
- new net PA_7: HBRIDGE.GND@6, U$9.PA7
- new net PA_8: Q8.G, R10.2, U$9.PA8
- new net PA_9: SERIAL.1, U$9.PA9
- new net PB_1: Q1.G, R19.2, U$9.PB1
- new net PB_10: HBRIDGE.GND@4, U$9.PB10
- new net PB_3: ENCODER.3, U$9.PB3
- new net PB_6: HBRIDGE.VS, U$9.PB6
- new net PC_0: Q6.E, R3.2, U$9.PC0
- new net PC_1: Q10.E, R4.2, U$9.PC1
- new net PC_2: Q11.E, R5.2, U$9.PC2
- new net PC_3: Q12.E, R6.2, U$9.PC3
- new net PC_4: ENCODER.10, U$9.PC4
- new net PC_7: HBRIDGE.IN1, U$9.PC7
- net 0.1MICROF: now also C2.2; no longer C2.1
- net 3.3V_NUCLEO: now also ENCODER.6, ENCODER.7; no longer ENCODER.4, JP2.4
- net 5V: now also IRE1.+; no longer HBRIDGE.VCC1, U$4.+
- net 5V_NUCLEO: now also HBRIDGE.IN2; no longer HBRIDGE.1-2EN, HBRIDGE.3-4EN
- net BAT: now also C2.1, HBRIDGE.OUT2, U$4.PIN2; no longer C2.2, S1.P
- net GND: now also C17.1, C17.2, ENCODER.12, HBRIDGE.GND@1, HBRIDGE.GND@2, HBRIDGE.IN3, HBRIDGE.OUT3, R11.1, R14.1, R16.1, R19.1, S1.3, SW.1; no longer HBRIDGE.GND1, HBRIDGE.GND3, HBRIDGE.GND4, JP2.1, R12.1, R2.1, R4.1, R6.1
- net MOTOR1A: now also ENCODER.4, HBRIDGE.GND@5; no longer ENCODER.5, HBRIDGE.4Y
- net MOTOR1B: now also ENCODER.2, HBRIDGE.EN2; no longer ENCODER.6, HBRIDGE.3Y
- net MOTOR2A: now also ENCODER.9, HBRIDGE.OUT1; no longer HBRIDGE.1Y, JP2.5
- net MOTOR2B: now also ENCODER.11, HBRIDGE.GND@3; no longer HBRIDGE.2Y, JP2.6
- net N$1: now also U$4.PIN3; no longer S1.S
- net N$10: now also R13.2; no longer R5.2
- net N$11: now also R13.1; no longer R5.1
- net N$12: now also R12.1; no longer R7.1
- net N$16: now also R7.2; no longer R11.2
- net N$17: now also R7.1; no longer R11.1
- net N$2: now also IRE1.-, R17.2; no longer R1.2, U$4.-
- net N$4: now also R17.1; no longer R1.1
- net N$5: now also R1.1, R2.1, R3.1, R4.1, R5.1, R6.1; no longer 1.8K.1, 1.8K1.1, 1.8K2.1, 1.8K3.1, 1.8K4.1, 1.8K5.1
- net N$6: now also R15.2; no longer R3.2
- net N$7: now also R15.1; no longer R3.1
- net N$9: now also R12.2; no longer R7.2
Other:
- note added: "IRE1 RIght Most"
- note added: "IRE2 Right Diagonal"
- note added: "IRE3 Right Front"
- note added: "IRE4 Left Front"
- note added: "IRE5 Left Diagonal"
- note added: "IRE6 Left Most"
- note added: "RX"
- note added: "TX"
- moved on the sheet: C1, C2, R1, R11, R12, R2, R3, R4, R5, R6, R7, R8

Commit message: changed power tags
Parts:
- added C18: 0.1uF, SparkFun:CAP0603-CAP
- Q1, Q2, Q3, Q7, Q8, Q9: value BS170 -> MOSFET-NCHANNELAO3404A; device transistor-small-signal:BS170 -> SparkFun-DiscreteSemi:MOSFET-NCHANNELAO3404A
- R10, R11, R14, R19, R8: value (none) -> 47K
- R16: value (none) -> 47k
Connections:
- removed net 3.3V_NUCLEO: ENCODER.6, ENCODER.7, Q10.C, Q11.C, Q12.C, Q4.C, Q5.C, Q6.C
- removed net 5V_NUCLEO: HBRIDGE.IN2
- removed net ASDF: S2.3
- removed net BOOT: S2.1, U$9.PB2
- new net BOOT0: S2.1, U$9.BOOT0
- new net BOOT1: U$9.PB2
- net 3.3V: now also ENCODER.6, ENCODER.7, Q10.C, Q11.C, Q12.C, Q4.C, Q5.C, Q6.C, U$9.VBAT, U$9.VDD_0, U$9.VDD_1, U$9.VDD_2, U$9.VDD_3
- net 5V: now also HBRIDGE.IN2, HBRIDGE.OUT2
- net BAT: no longer HBRIDGE.OUT2
- net GND: now also C18.1, C18.2, S2.3
- net N$11: now also Q1.D; no longer Q3.D
- net N$4: now also Q2.D; no longer Q1.D
- net N$7: now also Q3.D; no longer Q2.D
- net PA_3: now also Q1.G; no longer Q3.G
- net PA_6: now also Q3.G; no longer Q2.G
- net PB_1: now also Q2.G; no longer Q1.G
Other:
- moved on the sheet: C17, S1, S2

Commit message: fixed boot and nrst
still needs cap and resistor values
Parts:
- removed C17, C18: 0.1uF, SparkFun:CAP0603-CAP
- added C19, C20, C21, C22, C23: 100nF, SparkFun:CAP0603-CAP
- added R18, R20: 10k, SparkFun:RESISTOR0603-RES
Connections:
- new net BOOT2: R20.1
- net 0.1MICROF: no longer C1.1, U$5.EN
- net 3.3V: now also C19.1, C20.1, C21.1, C22.1, C23.1, R18.2, R20.2
- net 5V: now also C1.1, U$5.EN, U$5.IN
- net BAT: no longer U$5.IN
- net BOOT0: now also R18.1
- net GND: now also C19.2, C20.2, C21.2, C22.2, C23.2; no longer C17.1, C17.2, C18.1, C18.2
Other:
- moved on the sheet: C1, S2
